Commit message: Trying to add BlueROV URDF/Mesh into Visualizer

File: ros_ws/src/onboard/data_collection/urdf/bluerov2_sensors.urdf (robot description, URDF)
Before this commit: robot bluerov2, 4 links, 3 joints
Links:
- link base_link: geometry visual mesh filename=package://data_collection/meshes/bluerov2.dae scale=0.025 0.025 0.025

Commit message: Adjusting tf frame locations of ping360 and onboard camera

File: ros_ws/src/onboard/data_collection/urdf/bluerov2_sensors.urdf (robot description, URDF)
Before this commit: robot bluerov2, 4 links, 3 joints
Joints:
- joint camera_joint: origin xyz=-0.112 0 0.230 rpy=0 -0.05 0 -> xyz=0.0635 0 -0.1778 rpy=0 0 0
- joint sonar_joint: origin xyz=-0.18 0 -0.095 rpy=0 0 0 -> xyz=0.1143 -0.1143 0.1778 rpy=0 0 0

Commit message: Cleaned up visualization and corrected tf for who robot setup for future ping360 use in localization

File: ros_ws/src/onboard/data_collection/urdf/bluerov2_sensors.urdf (robot description, URDF)
Before this commit: robot bluerov2, 4 links, 3 joints
Links:
- added link sealbot; visual mesh filename=package://data_collection/meshes/Sealbot_Assembly.stl scale=0.001 0.001 0.001
- link base_link: geometry visual mesh filename=package://data_collection/meshes/bluerov2.dae scale=0.0254 0.0254 0.0254
- link sonar: geometry visual mesh filename=package://data_collection/meshes/ping360.stl
Joints:
- added joint sealbot_joint: type fixed, parent base_link, child sealbot, origin xyz=-0.0125 0 0.0725 rpy=0 0 0
- joint camera_joint: origin xyz=0.0635 0 -0.1778 rpy=0 0 0 -> xyz=0.0225 0 -0.1778 rpy=0 0 0
